Commit message: Sim setup with a single pipe rail surrounded by plants

File: humble_ws/src/iris_gazebo/urdf/plants.urdf (robot description, URDF)
Before this commit: robot plants, 4 links, 3 joints
Links:
- removed link world
Joints:
- removed joint plants_joint

File: humble_ws/src/iris_gazebo/urdf/rails.urdf (robot description, URDF)
Before this commit: robot rails, 2 links, 1 joints
Links:
- removed link world
Joints:
- removed joint rails_joint
