Commit message: Generated arm config for Kinova. Seems mostly functional but has some complain about opening display ':0'

File: humble_ws/install/kinova_arm/share/kinova_arm/description/urdf/GEN3_6DOF_VISION_URDF_ARM_V01.urdf (robot description, URDF)
Before this commit: robot GEN3_6DOF_VISION_URDF_ARM_V01, 11 links, 10 joints
Links:
- added link no_inertia_link
Joints:
- added joint joint_no_inertia: type fixed, parent no_inertia_link, child arm_base_link, origin xyz=0 0 0 rpy=0 0 0

Commit message: arm demo runs and executes plans!

File: humble_ws/install/kinova_arm/share/kinova_arm/description/urdf/GEN3_6DOF_VISION_URDF_ARM_V01.urdf (robot description, URDF)
Before this commit: robot GEN3_6DOF_VISION_URDF_ARM_V01, 12 links, 11 joints
Links:
- removed link no_inertia_link
Joints:
- removed joint joint_no_inertia
