Commit message: corrected arm position and made chassis_link the root link in URDF. Going to reload into moveit setup assistant and isaacsim, to ensure consistency between URDF models

File: humble_ws/install/antworker_description/share/antworker_description/description/combined/worker_with_arm.urdf (robot description, URDF)
Before this commit: robot antworker, 15 links, 14 joints
Links:
- removed link kbase_link
- added link base_link
Joints:
- removed joint robot_base_link_arm_base_link
- added joint arm_base_link_joint: type fixed, parent chassis_link, child arm_base_link, origin xyz=0.01 0.33 0.13 rpy=0 0 -1.57
- joint base_link_joint: child chassis_link -> base_link; origin xyz=0 0 0 rpy=0 0 0 -> xyz=0 0 0 rpy=0 0 -1.57; parent kbase_link -> chassis_link
