Commit message: Stripped down pipe rail model and now robot can get on and off of rail, and green wheels do not sink into rail

File: humble_ws/src/antworker_isaacsim_world/urdf/rails.urdf (robot description, URDF)
Before this commit: robot rails, 2 links, 1 joints
Links:
- removed link world
- link rails: geometry collision box size=50 0.15 0.15; collision box size=50 0.15 0.15
Joints:
- removed joint rails_joint

Commit message: Changed max joint speed for wheels to 600 degrees per second, so robot can hit 0.5 m/s now. Also changed pipe rail size to stop flanges from hitting ground

File: humble_ws/src/antworker_isaacsim_world/urdf/rails.urdf (robot description, URDF)
Before this commit: robot rails, 1 links, 0 joints
Links:
- link rails: mass 10000.0 -> None; geometry collision box size=50 0.1 0.1; collision box size=50 0.1 0.1
