Commit message: Even with 1 articulation controller, arm still wont move

File: humble_ws/src/antworker_description/description/combined/worker_with_arm.urdf (robot description, URDF)
Before this commit: robot antworker, 15 links, 14 joints
Links:
- removed link base_link
- added link kbase_link
Joints:
- joint base_link_joint: parent base_link -> kbase_link
- joint robot_base_link_arm_base_link: parent base_link -> kbase_link

Commit message: Added flanges to wheels

File: humble_ws/src/antworker_description/description/combined/worker_with_arm.urdf (robot description, URDF)
Before this commit: robot antworker, 15 links, 14 joints
Links:
- added link front_wheel_left_flange; collision cylinder length=0.05 radius=0.175; visual cylinder length=0.05 radius=0.175
- added link front_wheel_right_flange; collision cylinder length=0.05 radius=0.175; visual cylinder length=0.05 radius=0.175
- added link rear_wheel_left_flange; collision cylinder length=0.05 radius=0.175; visual cylinder length=0.05 radius=0.175
- added link rear_wheel_right_flange; collision cylinder length=0.05 radius=0.175; visual cylinder length=0.05 radius=0.175
Joints:
- added joint front_wheel_left_flange_joint: type fixed, parent front_wheel_link, child front_wheel_left_flange, origin xyz=0.375 0.0 rpy=0 0 0, axis 1 0 0
- added joint front_wheel_right_flange_joint: type fixed, parent front_wheel_link, child front_wheel_right_flange, origin xyz=-0.375 0.0 rpy=0 0 0, axis 1 0 0
- added joint rear_wheel_left_flange_joint: type fixed, parent rear_wheel_link, child rear_wheel_left_flange, origin xyz=0.375 0.0 rpy=0 0 0, axis 1 0 0
- added joint rear_wheel_right_flange_joint: type fixed, parent rear_wheel_link, child rear_wheel_right_flange, origin xyz=-0.375 0.0 rpy=0 0 0, axis 1 0 0

Commit message: Fixed base link / chassis link axis WRT chassis mesh. Only need base_link now, not chassis link as well. Need to add back the flanges.

File: humble_ws/src/antworker_description/description/combined/worker_with_arm.urdf (robot description, URDF)
Before this commit: robot antworker, 19 links, 18 joints
Links:
- removed link chassis_link
- removed link front_wheel_left_flange
- removed link front_wheel_right_flange
- removed link rear_wheel_left_flange
- removed link rear_wheel_right_flange
- link base_link: mass None -> 10; geometry collision mesh filename=package://antworker_description/description/base/meshes/ant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 scale=1.0 1.0 1.0; visual mesh filename=package://antworker_description/description/base/meshes/ant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 scale=1.0 1.0 1.0
Joints:
- removed joint base_link_joint
- removed joint front_wheel_left_flange_joint
- removed joint front_wheel_right_flange_joint
- removed joint rear_wheel_left_flange_joint
- removed joint rear_wheel_right_flange_joint
- joint arm_base_link_joint: origin xyz=0.01 0.33 0.13 rpy=0 0 -1.57 -> xyz=-0.33 0.01 0.13 rpy=0 0 -1.57; parent chassis_link -> base_link
- joint front_wheel_joint: axis 1 0 0 -> 0 0 1; origin xyz=0 0.395 -0.420 rpy=0 0 0 -> xyz=0.395 0 -0.420 rpy=1.57 0 0; parent chassis_link -> base_link
- joint rear_wheel_joint: axis 1 0 0 -> 0 0 1; origin xyz=0 -0.395 -0.420 rpy=0 0 0 -> xyz=-0.395 0 -0.420 rpy=1.57 0 0; parent chassis_link -> base_link

Commit message: Fixed cylinder wheel orientation so robot goes forward/backward as expected

File: humble_ws/src/antworker_description/description/combined/worker_with_arm.urdf (robot description, URDF)
Before this commit: robot antworker, 14 links, 13 joints
Joints:
- joint front_wheel_joint: origin xyz=0.395 0 -0.420 rpy=1.57 0 0 -> xyz=0.395 0 -0.420 rpy=-1.57 0 0
- joint rear_wheel_joint: origin xyz=-0.395 0 -0.420 rpy=1.57 0 0 -> xyz=-0.395 0 -0.420 rpy=-1.57 0 0

Commit message: Added flanges and decal back onto worker

File: humble_ws/src/antworker_description/description/combined/worker_with_arm.urdf (robot description, URDF)
Before this commit: robot antworker, 14 links, 13 joints
Links:
- added link decal; visual mesh filename=package://antworker_description/description/base/meshes/dec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 scale=0.01 0.01 0.01
- added link front_wheel_left_flange; collision cylinder length=0.05 radius=0.175; visual cylinder length=0.05 radius=0.175
- added link front_wheel_right_flange; collision cylinder length=0.05 radius=0.175; visual cylinder length=0.05 radius=0.175
- added link rear_wheel_left_flange; collision cylinder length=0.05 radius=0.175; visual cylinder length=0.05 radius=0.175
- added link rear_wheel_right_flange; collision cylinder length=0.05 radius=0.175; visual cylinder length=0.05 radius=0.175
Joints:
- added joint decal_fixed_joint: type fixed, parent base_link, child decal, origin xyz=0 0 0.15 rpy=0 0 0
- added joint front_wheel_left_flange_joint: type fixed, parent front_wheel_link, child front_wheel_left_flange, origin xyz=0 0 0.375 rpy=0 0 0
- added joint front_wheel_right_flange_joint: type fixed, parent front_wheel_link, child front_wheel_right_flange, origin xyz=0 0 -0.375 rpy=0 0 0
- added joint rear_wheel_left_flange_joint: type fixed, parent rear_wheel_link, child rear_wheel_left_flange, origin xyz=0 0 0.375 rpy=0 0 0
- added joint rear_wheel_right_flange_joint: type fixed, parent rear_wheel_link, child rear_wheel_right_flange, origin xyz=0 0 -0.375 rpy=0 0 0

Commit message: Took xy tolerance down in followpath and goal checker, robot is now hitting 99%+ accuracy, albeit with perfectct odometry from sim

File: humble_ws/src/antworker_description/description/combined/worker_with_arm.urdf (robot description, URDF)
Before this commit: robot antworker, 19 links, 18 joints
Joints:
- joint decal_fixed_joint: origin xyz=0 0 0.15 rpy=0 0 0 -> xyz=0 0 0 rpy=0 0 0

File: humble_ws/src/antworker_isaacsim_world/urdf/rails.urdf (robot description, URDF)
Before this commit: robot rails, 1 links, 0 joints
Links:
- link rails: geometry collision box size=60 0.1 0.1; collision box size=60 0.1 0.1
